Commit message: Updating repo

File: grasp01_description/urdf/grasp01_description.urdf (robot description, URDF)
Before this commit: robot grasp01_description, 8 links, 7 joints
Joints:
- joint ee_joint: limit lower=-1.0472 upper=1.0472 effort=0 velocity=0 -> lower=-1.0472 upper=1.0472 effort=0 velocity=1.0
- joint joint_1: limit lower=-1.57 upper=1.57 effort=0 velocity=0 -> lower=-1.57 upper=1.57 effort=0 velocity=1.0
- joint joint_2: limit lower=-1.57 upper=1.57 effort=0 velocity=0 -> lower=-1.57 upper=1.57 effort=0 velocity=1.0
- joint joint_3: limit lower=-1.57 upper=1.57 effort=0 velocity=0 -> lower=-1.57 upper=1.57 effort=0 velocity=1.0
- joint joint_4: limit lower=-1.57 upper=1.57 effort=0 velocity=0 -> lower=-1.57 upper=1.57 effort=0 velocity=1.0
- joint joint_5: limit lower=-1.57 upper=1.57 effort=0 velocity=0 -> lower=-1.57 upper=1.57 effort=0 velocity=1.0

File: grasp01_moveit2/config/grasp01_description.ros2_control.xacro (robot description, xacro)
@@ -1,70 +1,64 @@
 <?xml version="1.0"?>
 <robot xmlns:xacro="http://www.ros.org/wiki/xacro">
-    <xacro:macro name="grasp01_description_ros2_control" params="name initial_positions_file">
-        <xacro:property name="initial_positions" value="${load_yaml(initial_positions_file)['initial_positions']}"/>
+    <xacro:macro name="grasp01_description_ros2_control" params="name initial_positions ifname cycle_time timeout">
+        <!-- No need to load YAML here; initial_positions is already a dictionary -->
         <ros2_control name="${name}" type="system">
             <hardware>
-                <!-- By default, set up controllers for simulation. This won't work on real hardware -->
-                <plugin>mock_components/GenericSystem</plugin>
+                <!-- Use the custom hardware interface for the real Grasp01 arm -->
+                <plugin>grasp01_hardware/Grasp01HardwareInterface</plugin>
+                <!-- Hardware-specific parameters -->
+                <param name="ifname">${ifname}</param>          <!-- CAN interface name, e.g., "can0" -->
+                <param name="cycle_time">${cycle_time}</param>  <!-- Control cycle time in ms, e.g., "1" -->
+                <param name="timeout">${timeout}</param>        <!-- Actuator timeout in ms, e.g., "0" -->
             </hardware>
             <joint name="joint_1">
                 <command_interface name="position"/>
-                <command_interface name="velocity"/>
-                <command_interface name="effort"/>
                 <state_interface name="position">
-                  <param name="initial_value">${initial_positions['joint_1']}</param>
+                    <param name="initial_value">${initial_positions['joint_1']}</param>
                 </state_interface>
-                <state_interface name="velocity"/>
-                <state_interface name="effort"/>
+                <!-- Joint-specific parameters -->
+                <param name="actuator_id">1</param>
+                <param name="torque_constant">0.1</param>
             </joint>
             <joint name="joint_2">
                 <command_interface name="position"/>
-                <command_interface name="velocity"/>
-                <command_interface name="effort"/>
                 <state_interface name="position">
-                  <param name="initial_value">${initial_positions['joint_2']}</param>
+                    <param name="initial_value">${initial_positions['joint_2']}</param>
                 </state_interface>
-                <state_interface name="velocity"/>
-                <state_interface name="effort"/>
+                <param name="actuator_id">2</param>
+                <param name="torque_constant">0.1</param>
             </joint>
             <joint name="joint_3">
                 <command_interface name="position"/>
-                <command_interface name="velocity"/>
-                <command_interface name="effort"/>
                 <state_interface name="position">
-                  <param name="initial_value">${initial_positions['joint_3']}</param>
+                    <param name="initial_value">${initial_positions['joint_3']}</param>
                 </state_interface>
-                <state_interface name="velocity"/>
-                <state_interface name="effort"/>
+                <param name="actuator_id">3</param>
+                <param name="torque_constant">0.1</param>
             </joint>
             <joint name="joint_4">
                 <command_interface name="position"/>
-                <command_interface name="velocity"/>
-                <command_interface name="effort"/>
                 <state_interface name="position">
-                  <param name="initial_value">${initial_positions['joint_4']}</param>
+                    <param name="initial_value">${initial_positions['joint_4']}</param>
                 </state_interface>
-                <state_interface name="velocity"/>
-                <state_interface name="effort"/>
+                <param name="actuator_id">4</param>
+                <param name="torque_constant">0.1</param>
             </joint>
             <joint name="joint_5">
                 <command_interface name="position"/>
-                <command_interface name="velocity"/>
-                <command_interface name="effort"/>
                 <state_interface name="position">
-                  <param name="initial_value">${initial_positions['joint_5']}</param>
+                    <param name="initial_value">${initial_positions['joint_5']}</param>
                 </state_interface>
-                <state_interface name="velocity"/>
-                <state_interface name="effort"/>
+                <param name="actuator_id">5</param>
+                <param name="torque_constant">0.1</param>
             </joint>
             <joint name="ee_joint">
                 <command_interface name="position"/>
-                <command_interface name="velocity"/>
-                <command_interface name="effort"/>
                 <state_interface name="position">
-                  <param name="initial_value">${initial_positions['ee_joint']}</param>
+                    <param name="initial_value">${initial_positions['ee_joint']}</param>
                 </state_interface>
-                <state_interface name="velocity"/>
-                <state_interface name="effort"/>
+                <param name="actuator_id">6</param>
+                <param name="torque_constant">0.1</param>
+                <param name="max_velocity">1.0</param>
             </joint>
         </ros2_control>

File: grasp01_moveit2/config/grasp01_description.urdf.xacro (robot description, xacro)
@@ -1,9 +1,24 @@
 <?xml version="1.0"?>
 <robot xmlns:xacro="http://www.ros.org/wiki/xacro" name="grasp01_description">
-    <xacro:arg name="initial_positions_file" default="initial_positions.yaml" />
+    <!-- Define arguments -->
+    <xacro:arg name="ifname" default="can0" />
+    <xacro:arg name="cycle_time" default="1" />
+    <xacro:arg name="timeout" default="0" />
+    <!-- Define the argument with a default value -->
+    <xacro:arg name="initial_positions_file" default="$(find grasp01_moveit2)/config/initial_positions.yaml" />
+    <!-- Explicitly set the file path as a property -->
+    <xacro:property name="initial_positions_file_path" value="$(arg initial_positions_file)" />
+    <!-- Load the YAML file using the property -->
+    <xacro:property name="initial_positions" value="${xacro.load_yaml(initial_positions_file_path)['initial_positions']}" scope="global" />
     <!-- Import grasp01_description urdf file -->
     <xacro:include filename="$(find grasp01_description)/urdf/grasp01_description.urdf" />
     <!-- Import control_xacro -->
     <xacro:include filename="grasp01_description.ros2_control.xacro" />
-    <xacro:grasp01_description_ros2_control name="FakeSystem" initial_positions_file="$(arg initial_positions_file)"/>
+    <!-- Call the ROS2 control macro with the loaded YAML data -->
+    <xacro:grasp01_description_ros2_control
+        name="Grasp01Control"
+        initial_positions="${initial_positions}"
+        ifname="$(arg ifname)"
+        cycle_time="$(arg cycle_time)"
+        timeout="$(arg timeout)"/>
 </robot>

Commit message: Adding new files and packages

File: grasp01_description/urdf/grasp01_description.urdf (robot description, URDF)
Before this commit: robot grasp01_description, 8 links, 7 joints
Joints:
- joint joint_1: origin xyz=0.38681 -0.060538 -0.10561 rpy=-0.01389 0.039152 0.010785 -> xyz=0.0 0.0 0.0 rpy=0.0 0.0 0.0

File: grasp01_gazebo/urdf/grasp01_gazebo.ros2_control.xacro (robot description, xacro)
@@ -1,11 +1,8 @@
 <?xml version="1.0"?>
 <robot xmlns:xacro="http://www.ros.org/wiki/xacro">
-  <xacro:macro name="grasp01_description_ros2_control" params="name initial_positions ifname cycle_time timeout">
-    <ros2_control name="${name}" type="system">
+  <xacro:macro name="grasp01_gazebo_ros2_control" params="name initial_positions">
+    <ros2_control name="IgnitionSystem" type="system">
       <hardware>
-        <plugin>grasp01_hardware/Grasp01HardwareInterface</plugin>
-        <param name="ifname">${ifname}</param>          <!-- CAN interface name, e.g., "can0" -->
-        <param name="cycle_time">${cycle_time}</param>  <!-- Control cycle time in ms, e.g., "1" -->
-        <param name="timeout">${timeout}</param>        <!-- Actuator timeout in ms, e.g., "0" -->
+        <plugin>ign_ros2_control/IgnitionSystem</plugin>
       </hardware>
       <joint name="joint_1">
@@ -13,11 +10,9 @@
         <command_interface name="effort"/>
         <command_interface name="velocity"/>
-        <state_interface name="effort"/>
         <state_interface name="position">
           <param name="initial_value">${initial_positions['joint_1']}</param>
         </state_interface>
-        <!-- Joint-specific parameters -->
-        <param name="actuator_id">1</param>
-        <param name="torque_constant">0.1</param>
+        <state_interface name="velocity"/>
+        <state_interface name="effort"/>
       </joint>
       <joint name="joint_2">
@@ -25,10 +20,9 @@
         <command_interface name="effort"/>
         <command_interface name="velocity"/>
-        <state_interface name="effort"/>
         <state_interface name="position">
           <param name="initial_value">${initial_positions['joint_2']}</param>
         </state_interface>
-        <param name="actuator_id">2</param>
-        <param name="torque_constant">0.1</param>
+        <state_interface name="velocity"/>
+        <state_interface name="effort"/>
       </joint>
       <joint name="joint_3">
@@ -36,10 +30,9 @@
         <command_interface name="effort"/>
         <command_interface name="velocity"/>
-        <state_interface name="effort"/>
         <state_interface name="position">
           <param name="initial_value">${initial_positions['joint_3']}</param>
         </state_interface>
-        <param name="actuator_id">3</param>
-        <param name="torque_constant">0.1</param>
+        <state_interface name="velocity"/>
+        <state_interface name="effort"/>
       </joint>
       <joint name="joint_4">
@@ -47,10 +40,9 @@
         <command_interface name="effort"/>
         <command_interface name="velocity"/>
-        <state_interface name="effort"/>
         <state_interface name="position">
           <param name="initial_value">${initial_positions['joint_4']}</param>
         </state_interface>
-        <param name="actuator_id">4</param>
-        <param name="torque_constant">0.1</param>
+        <state_interface name="velocity"/>
+        <state_interface name="effort"/>
       </joint>
       <joint name="joint_5">
@@ -58,10 +50,9 @@
         <command_interface name="effort"/>
         <command_interface name="velocity"/>
-        <state_interface name="effort"/>
         <state_interface name="position">
           <param name="initial_value">${initial_positions['joint_5']}</param>
         </state_interface>
-        <param name="actuator_id">5</param>
-        <param name="torque_constant">0.1</param>
+        <state_interface name="velocity"/>
+        <state_interface name="effort"/>
       </joint>
       <joint name="ee_joint">
@@ -69,11 +60,9 @@
         <command_interface name="effort"/>
         <command_interface name="velocity"/>
-        <state_interface name="velocity"/>
-        <state_interface name="effort"/>
         <state_interface name="position">
           <param name="initial_value">${initial_positions['ee_joint']}</param>
         </state_interface>
-        <param name="actuator_id">6</param>
-        <param name="torque_constant">0.1</param>
+        <state_interface name="velocity"/>
+        <state_interface name="effort"/>
       </joint>
     </ros2_control>

Commit message: adding new files

File: grasp01_description/urdf/grasp01_description.urdf (robot description, URDF)
Before this commit: robot grasp01_description, 8 links, 7 joints
Links:
- link base_link: mass 2.2301 -> 1.3236
- link ee_link: mass 0.21749 -> 0.27187
- link link_1: mass 0.252 -> 1.215
- link link_2: mass 0.32937 -> 1.311
- link link_3: mass 0.252 -> 1.215
- link link_4: mass 1.0139 -> 1.33
- link link_5: mass 0.60833 -> 1.088
Joints:
- joint ee_joint: limit lower=-1.0472 upper=1.0472 effort=0 velocity=1.0 -> lower=-1.0472 upper=1.0472 effort=0 velocity=0.0; origin xyz=0.23695 -0.018844 0.029243 rpy=-0.01298 -0.070854 0.046424 -> xyz=0.23586 -0.018782 0.029068 rpy=-0.010928 -0.060804 0.039747
- joint joint_1: limit lower=-1.57 upper=1.57 effort=0 velocity=1.0 -> lower=-1.57 upper=1.57 effort=0 velocity=0.0
- joint joint_2: axis 0.99871 0 0.050703 -> -0.99871 0 0.050703; limit lower=-1.57 upper=1.57 effort=0 velocity=1.0 -> lower=-1.57 upper=1.57 effort=0 velocity=0.0; origin xyz=0 -0.093789 0 rpy=-0.032166 -2.6262E-05 -0.0016327 -> xyz=0 -0.096506 0 rpy=-0.050536 -6.4814E-05 -0.0025645
- joint joint_3: axis 0.050641 0.049454 -0.99749 -> 0.050641 0.049454 0.99749; limit lower=-1.57 upper=1.57 effort=0 velocity=1.0 -> lower=-1.57 upper=1.57 effort=0 velocity=0.0; origin xyz=0.0091425 0.0094159 -0.18995 rpy=-0.00021387 -0.00020798 0.0042041 -> xyz=0.0090236 0.0092998 -0.1876 rpy=-0.0056952 -0.0049964 0.10683
- joint joint_4: limit lower=-1.57 upper=1.57 effort=0 velocity=1.0 -> lower=-1.57 upper=1.57 effort=0 velocity=0.0; origin xyz=0.0049917 0.0048747 -0.098324 rpy=2.506 1.3895 2.5101 -> xyz=0.00506 0.0049414 -0.099668 rpy=2.2009 1.442 2.2049
- joint joint_5: axis 0.98605 -0.055724 0.15683 -> -0.98605 -0.055724 0.15683; limit lower=-1.57 upper=1.57 effort=0 velocity=1.0 -> lower=-1.57 upper=1.57 effort=0 velocity=0.0; origin xyz=0.13582 -0.0071752 0.021623 rpy=0.47438 -0.0435 0.066585 -> xyz=0.13691 -0.0072371 0.021798 rpy=-2.4329 -0.24294 -0.20316
- joint world_to_base: origin xyz=0 0 1.2 rpy=0 0 0 -> xyz=0 0 2.0 rpy=0 0 0

File: grasp01_gazebo/urdf/grasp01_gazebo.ros2_control.xacro (robot description, xacro)
@@ -2,12 +2,12 @@
 <robot xmlns:xacro="http://www.ros.org/wiki/xacro">
   <xacro:macro name="grasp01_gazebo_ros2_control" params="name initial_positions">
-    <ros2_control name="IgnitionSystem" type="system">
+    <ros2_control name="GazeboSystem" type="system">
       <hardware>
-        <plugin>ign_ros2_control/IgnitionSystem</plugin>
+        <plugin>gazebo_ros2_control/GazeboSystem</plugin>
       </hardware>
       <joint name="joint_1">
-        <command_interface name="position"/>
+        <!-- <command_interface name="position"/> -->
         <command_interface name="effort"/>
-        <command_interface name="velocity"/>
+        <!-- <command_interface name="velocity"/> -->
         <state_interface name="position">
           <param name="initial_value">${initial_positions['joint_1']}</param>
@@ -17,7 +17,7 @@
       </joint>
       <joint name="joint_2">
-        <command_interface name="position"/>
+        <!-- <command_interface name="position"/> -->
         <command_interface name="effort"/>
-        <command_interface name="velocity"/>
+        <!-- <command_interface name="velocity"/> -->
         <state_interface name="position">
           <param name="initial_value">${initial_positions['joint_2']}</param>
@@ -27,7 +27,7 @@
       </joint>
       <joint name="joint_3">
-        <command_interface name="position"/>
+        <!-- <command_interface name="position"/> -->
         <command_interface name="effort"/>
-        <command_interface name="velocity"/>
+        <!-- <command_interface name="velocity"/> -->
         <state_interface name="position">
           <param name="initial_value">${initial_positions['joint_3']}</param>
@@ -37,7 +37,7 @@
       </joint>
       <joint name="joint_4">
-        <command_interface name="position"/>
+        <!-- <command_interface name="position"/> -->
         <command_interface name="effort"/>
-        <command_interface name="velocity"/>
+        <!-- <command_interface name="velocity"/> -->
         <state_interface name="position">
           <param name="initial_value">${initial_positions['joint_4']}</param>
@@ -47,7 +47,7 @@
       </joint>
       <joint name="joint_5">
-        <command_interface name="position"/>
+        <!-- <command_interface name="position"/> -->
         <command_interface name="effort"/>
-        <command_interface name="velocity"/>
+        <!-- <command_interface name="velocity"/> -->
         <state_interface name="position">
           <param name="initial_value">${initial_positions['joint_5']}</param>
@@ -57,7 +57,7 @@
       </joint>
       <joint name="ee_joint">
-        <command_interface name="position"/>
+        <!-- <command_interface name="position"/> -->
         <command_interface name="effort"/>
-        <command_interface name="velocity"/>
+        <!-- <command_interface name="velocity"/> -->
         <state_interface name="position">
           <param name="initial_value">${initial_positions['ee_joint']}</param>

File: grasp01_gazebo/urdf/grasp01_gazebo.urdf.xacro (robot description, xacro)
@@ -9,5 +9,5 @@
     <!-- Import grasp01_description urdf file -->
     <xacro:include filename="$(find grasp01_description)/urdf/grasp01_description.urdf" />
-    <!-- Import control_xacro -->
+    <!-- Import control_xacro (optional, if still needed) -->
     <xacro:include filename="$(find grasp01_gazebo)/urdf/grasp01_gazebo.ros2_control.xacro" />
     <!-- Call the ROS2 control macro with minimal parameters for simulation -->
@@ -15,11 +15,20 @@
         name="Grasp01Control"
         initial_positions="${initial_positions}" />
-    <!-- Gazebo Ionic ROS2 Control Plugin for Simulation -->
-    <gazebo>
-      <plugin filename="ign_ros2_control-system" name="ign_ros2_control::IgnitionROS2ControlPlugin">
-        <robot_param>robot_description</robot_param>
-        <robot_param_node>robot_state_publisher</robot_param_node>
-        <parameters>$(find grasp01_gazebo)/config/ros2_gazebi_controllers.yaml</parameters>
-      </plugin>
-    </gazebo>
+    <!-- Gazebo Classic ROS2 Control Plugin -->
+     <!-- Add gazebo_ros2_control plugin -->
+  <gazebo>
+    <plugin name="gazebo_ros2_control" filename="libgazebo_ros2_control.so">
+      <robotParam>robot_description</robotParam>
+      <robotParamName>robot_description</robotParamName>
+      <commandInterfaces>
+        <interface>effort</interface>
+      </commandInterfaces>
+      <stateInterfaces>
+        <interface>position</interface>
+        <interface>velocity</interface>
+        <interface>effort</interface>
+      </stateInterfaces>
+      <parameters>$(find grasp01_gazebo)/config/ros2_gazebo_controllers.yaml</parameters>
+    </plugin>
+  </gazebo>
 </robot>
